Commit message: Added dockerfile for running navigation stack

File: roombot/roombot_description/urdf/roombot_rs.urdf.xacro (robot description, xacro)
@@ -7,9 +7,9 @@
 	<xacro:arg name="use_mesh" default="true" />
 	<xacro:include filename="$(find realsense2_description)/urdf/_d435.urdf.xacro" />
-	<xacro:create_base wheel_seperation="0.235" base_diameter="0.3485">
-		<mesh filename="package://create_description/meshes/create_2.dae" />
+	<xacro:create_base wheel_separation="0.235" base_diameter="0.3485">
+		<mesh filename="$(find create_description)/meshes/create_2.dae" />
 	</xacro:create_base>
-	<xacro:sensor_d435 parent="base_link" use_nominal_extrinsics="$(arg use_nominal_extrinsics)" add_plug="$(arg add_plug)" use_mesh="$(arg use_mesh)">
-		<origin xyz="0 0 0" rpy="0 0 0"/>
+	<xacro:sensor_d435 parent="base_footprint" use_nominal_extrinsics="$(arg use_nominal_extrinsics)" add_plug="$(arg add_plug)" use_mesh="$(arg use_mesh)">
+		<origin xyz="0.155 0 0.155" rpy="0 0 0"/>
 	</xacro:sensor_d435>
 </robot>
